File: radio_sx1280/sx1280.kicad_pcb (KiCad board)
At the start: 4 copper layers, 16 x 17 mm, 32 parts, among them J1 Conn_01x01, J10 Conn_01x01, J11 Conn_01x01, J12 Conn_01x01, J13 Conn_01x01, J14 Conn_01x01, J15 Conn_01x01, J16 Conn_01x01, J2 Conn_01x01, J3 Conn_01x01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

Commit message: added layer markings and annotated silk screen and gave 0.254mm clearance b/t inner layer copper plane and bord edge cut
Other:
- board text added: "SX1280 2.4 GHz Kustin"
- board text removed: "SX1280 2.4 GHz"
Changed lines of the file:
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@@
     (effects (font (size 0.508 0.508) (thickness 0.1016)) (justify right))
   )
-  (gr_text "SX1280\n2.4 GHz" (at 107.442 105.537) (layer "F.Mask")
+  (gr_text "SX1280\n2.4 GHz\nKustin" (at 107.442 106.934) (layer "F.Mask")
     (effects (font (size 0.762 0.762) (thickness 0.1905)))
+  )
+  (dimension (type aligned) (layer "In1.Cu")
+    (pts (xy 115.062 114.046) (xy 114.808 114.046))
+    (height -12.192)
+    (gr_text "0.2540 mm" (at 114.935 125.613) (layer "In1.Cu")
+      (effects (font (size 0.5 0.5) (thickness 0.3)))
+    )
+    (format (units 3) (units_format 1) (precision 4))
+    (style (thickness 0.05) (arrow_length 0.1) (text_position_mode 0) (extension_height 0.58642) (extension_offset 0.5) keep_text_aligned)
+  )
+  (dimension (type aligned) (layer "In1.Cu")
+    (pts (xy 109.474 103.632) (xy 109.474 103.886))
+    (height -10.668)
+    (gr_text "0.2540 mm" (at 119.517 103.759 90) (layer "In1.Cu")
+      (effects (font (size 0.5 0.5) (thickness 0.3)) (justify right))
+    )
+    (format (units 3) (units_format 1) (precision 4))
+    (style (thickness 0.05) (arrow_length 0.1) (text_position_mode 0) (extension_height 0.58642) (extension_offset 0.5) keep_text_aligned)
   )
   (segment (start 107.137153 109.385053) (end 107.022947 109.385053) (width 0.508) (layer "F.Cu") (net 1))
@@
     )
   )
-  (zone (net 0) (net_name "") (layers "F.Cu" "In1.Cu" "In2.Cu" "B.Cu") (name "layerNumber") (hatch edge 0.508)
+  (zone (net 0) (net_name "") (layers "F.Cu" "In1.Cu") (name "layerNumber2") (hatch edge 0.508)
+    (connect_pads (clearance 0))
+    (min_thickness 0.254)
+    (keepout (tracks not_allowed) (vias not_allowed) (pads not_allowed ) (copperpour not_allowed) (footprints allowed))
+    (fill (thermal_gap 0.508) (thermal_bridge_width 0.508))
+    (polygon
+      (pts
+        (xy 106.426 105.41)
+        (xy 104.902 105.41)
+        (xy 104.902 104.14)
+        (xy 106.426 104.14)
+      )
+    )
+  )
+  (zone (net 3) (net_name "GND") (layer "In1.Cu") (hatch edge 0.508)
+    (connect_pads (clearance 0.127))
+    (min_thickness 0.127) (filled_areas_thickness no)
+    (fill yes (thermal_gap 0.127) (thermal_bridge_width 0.1524))
+    (polygon
+      (pts
+        (xy 99.314 103.886)
+        (xy 114.808 103.886)
+        (xy 114.808 120.396)
+        (xy 99.314 120.396)
+      )
+    )
+  )
+  (zone (net 0) (net_name "") (layers "In2.Cu" "B.Cu") (name "layerNumber3") (hatch edge 0.508)
     (connect_pads (clearance 0))
     (min_thickness 0.254)
@@
       )
     )
-  )
-  (zone (net 0) (net_name "") (layers "F.Cu" "In1.Cu" "In2.Cu" "B.Cu") (name "layerNumber") (hatch edge 0.508)
-    (connect_pads (clearance 0))
-    (min_thickness 0.254)
-    (keepout (tracks not_allowed) (vias not_allowed) (pads not_allowed ) (copperpour not_allowed) (footprints allowed))
-    (fill (thermal_gap 0.508) (thermal_bridge_width 0.508))
-    (polygon
-      (pts
-        (xy 106.426 105.156)
-        (xy 104.902 105.156)
-        (xy 104.902 103.886)
-        (xy 106.426 103.886)
-      )
-    )
-  )
-  (zone (net 3) (net_name "GND") (layer "In1.Cu") (hatch edge 0.508)
-    (connect_pads (clearance 0.127))
-    (min_thickness 0.127) (filled_areas_thickness no)
-    (fill yes (thermal_gap 0.127) (thermal_bridge_width 0.1524))
-    (polygon
-      (pts
-        (xy 99.06 103.632)
-        (xy 115.062 103.632)
-        (xy 115.062 120.65)
-        (xy 99.06 120.65)
-      )
-    )
